Commit message: holonomic bug control (quite good results) nonholonomic and castor bug control (inertia-related issues)

File: src/m2wr_description/urdf/m2wr.xacro (robot description, xacro)
@@ -60,5 +60,5 @@
     <!-- caster front -->
     <collision name="caster_front_collision">
-      <origin rpy=" 0 0 0" xyz="0.35 0 -0.05"/>
+      <origin rpy=" 0 0 0" xyz="0.35 0 -0.15"/>
       <geometry>
         <sphere radius="0.05"/>
@@ -76,5 +76,5 @@
     </collision>
     <visual name="caster_front_visual">
-      <origin rpy=" 0 0 0" xyz="0.2 0 -0.05"/>
+      <origin rpy=" 0 0 0" xyz="0.2 0 -0.15"/>
       <geometry>
         <sphere radius="0.05"/>

File: src/node_counting_alg/urdf/robot_castor.xacro (robot description, xacro)
@@ -1,4 +1,4 @@
 <?xml version="1.0"?>
-<robot name="nonhol"
+<robot name="castor"
 	xmlns:xacro="http://www.ros.org/wiki/xacro">
 	<!-- Included files -->
@@ -7,13 +7,11 @@
 	<!-- _______________________________________________________ -->
 	<!-- Create robot's base_link -->
-	<xacro:base_link name="base_link" size_x = "0.4" size_y = "0.2" size_z = "0.1" mass="5" />
+	<xacro:base_link name="base_link" size_x = "0.4" size_y = "0.2" size_z = "0.1" mass="5"/>
 	<!-- Create wheels -->
-	<xacro:wheel_link name="link_lfront_wheel" mass = "0.2"/>
-	<xacro:wheel_joint name="joint_lfront_wheel" child="link_lfront_wheel" origin_xyz="0.15 0.15 0"/>
-	<xacro:wheel_link name="link_rfront_wheel" mass = "0.2"/>
-	<xacro:wheel_joint name="joint_rfront_wheel" child="link_rfront_wheel" origin_xyz="0.15 -0.15 0"/>
-	<xacro:wheel_link name="link_lrear_wheel" mass = "0.2"/>
+	<xacro:wheel_link name="link_front_wheel" mass="0.2"/>
+	<xacro:omniwheel_joint name="joint_front_wheel" child="link_front_wheel" origin_xyz="0.15 0 0"/>
+	<xacro:wheel_link name="link_lrear_wheel" mass="0.2"/>
 	<xacro:wheel_joint name="joint_lrear_wheel" child="link_lrear_wheel" origin_xyz="-0.15 0.15 0"/>
-	<xacro:wheel_link name="link_rrear_wheel" mass = "0.2" />
+	<xacro:wheel_link name="link_rrear_wheel" mass="0.2"/>
 	<xacro:wheel_joint name="joint_rrear_wheel" child="link_rrear_wheel" origin_xyz="-0.15 -0.15 0"/>
 	<!-- Create camera -->
